File: drone.kicad_sch (KiCad schematic)
At the start: 0 parts

Commit message: Added sensors and mcu
Parts:
- added J1: Battery-Banana-Plug-Connector, symbol Connector_Generic:Conn_01x02
- added J10: GPIO7 TH, symbol Connector_Generic:Conn_01x01
- added J11, J12, J13, J14, J15, J16, J17, J18, J19, J20, J8: Conn_01x01, symbol Connector_Generic:Conn_01x01
- added J2: AF-MPM3610-Converter, Adafruit MPM3610:1X04_ROUND, symbol Adafruit MPM3610-eagle-import:HEADER-1X4ROUND
- added J21: GPIO9_TH, symbol Connector_Generic:Conn_01x01
- added J22: GPIO8 TH, symbol Connector_Generic:Conn_01x01
- added J3: ESC_1, symbol Connector_Generic:Conn_01x01
- added J4: ESC_2, symbol Connector_Generic:Conn_01x01
- added J5, J6: ESC_3, symbol Connector_Generic:Conn_01x01
- added J7: VCC_MCU_Sensors, symbol Connector_Generic:Conn_01x01
- added J9: GPIO44 TH, symbol Connector_Generic:Conn_01x01
- added S1: AF-QMC5883P-Magnetometer, Adafruit QMC5883P Magnetometer:1X05_ROUND_70, symbol Adafruit QMC5883P Magnetometer-eagle-import:HEADER-1X570MIL
- added S2: AF-BMP280-Barometer, Adafruit BMP280:1X07_ROUND_70, symbol Adafruit BMP280-eagle-import:HEADER-1X770MIL
- added S3: AF-MPU6050-Accel/Gyro, Adafruit MPU6050:1X06_ROUND_70, symbol Adafruit MPU6050-eagle-import:HEADER-1X670MIL
- added S4: AF-MPU6050-Accel/Gyro, Adafruit MPU6050:1X06_ROUND, symbol Adafruit MPU6050-eagle-import:HEADER-1X6ROUND
- added U1, U2: ESP32-S3, symbol Adafruit BMP280-eagle-import:HEADER-1X770MIL
Connections:
- new net: J14.1 (Pin_1), S4.4
- new net 3Vo: S1.2, S2.2, S3.2
- new net 5VIN: U1.1
- new net AD0: J11.1 (Pin_1), S4.1
- new net CLKIN: J15.1 (Pin_1), S4.5
- new net CS_5V: S2.7
- new net EN: J2.1
- new net FSYNC_IN: J12.1 (Pin_1), S4.2
- new net GND: J1.2 (Pin_2), J2.4, S1.3, S2.3, S3.3, S4.6, U1.2
- new net GPIO1: J16.1 (Pin_1), U2.1
- new net GPIO2: J17.1 (Pin_1), U2.2
- new net GPIO3: J18.1 (Pin_1), U2.3
- new net GPIO4: J19.1 (Pin_1), U2.4
- new net GPIO43: J20.1 (Pin_1), S1.4, S2.4, S3.4, U2.6, U2.7
- new net GPIO44: J9.1 (Pin_1), U1.7
- new net GPIO7: J10.1 (Pin_1), U1.6
- new net GPIO8: J22.1 (Pin_1), U1.5
- new net GPIO9: J21.1 (Pin_1), U1.4
- new net INT: S3.6
- new net SCL_EXT: J13.1 (Pin_1), S4.3
- new net SDA: S1.5, S2.6, S3.5, U2.5
- new net SDO/ADR_3V: S2.5
- new net VBat: J1.1 (Pin_1), J2.2, J3.1 (Pin_1), J4.1 (Pin_1), J5.1 (Pin_1), J6.1 (Pin_1)
- new net VCC_3V3: J2.3, J8.1 (Pin_1)
- new net VCC_3V3_MCU: J7.1 (Pin_1), S1.1, S2.1, S3.1, U1.3

Commit message: Initial commit 2
Parts:
- removed J3: ESC_1, symbol Connector_Generic:Conn_01x01
- removed J4: ESC_2, symbol Connector_Generic:Conn_01x01
- removed J5: ESC_3, symbol Connector_Generic:Conn_01x01
- added J18, J20, J27, J28, J29, J8, J9: Conn_01x01, symbol Connector_Generic:Conn_01x01
- added J2: Conn_ESC_PWR_1, symbol Connector_Generic:Conn_01x02
- added J3: Conn_ESC_PWR_2, symbol Connector_Generic:Conn_01x02
- added J30: Conn_SCL_Sensors, symbol Connector_Generic:Conn_01x01
- added J31: Conn_SDA_Sensors, symbol Connector_Generic:Conn_01x01
- added J32: Conn_ESC_SIG_1, symbol Connector_Generic:Conn_01x02
- added J33: Conn_ESC_SIG_2, symbol Connector_Generic:Conn_01x02
- added J34: Conn_ESC_SIG_3, symbol Connector_Generic:Conn_01x02
- added J35: Conn_ESC_SIG_4, symbol Connector_Generic:Conn_01x02
- added J36: Conn_MCUtoESC_1, symbol Connector_Generic:Conn_01x01
- added J37: Conn_MCUtoESC_2, symbol Connector_Generic:Conn_01x01
- added J38: Conn_MCUtoESC_3, symbol Connector_Generic:Conn_01x01
- added J39: Conn_MCUtoESC_4, symbol Connector_Generic:Conn_01x01
- added J4: Conn_ESC_PWR_3, symbol Connector_Generic:Conn_01x02
- added J5: Conn_ESC_PWR_4, symbol Connector_Generic:Conn_01x02
- J1: value Battery-Banana-Plug-Connector -> Conn_Lipo_Battery
- J21: renamed from J7; value VCC_MCU_Sensors -> Conn_01x01
- J6: value ESC_3 -> Conn_01x01
- U1: value ESP32-S3 -> ----Seeed-XIAO-ESP32-S3-Module----
- renumbered J21 to J10, J22 to J11, J10 to J12, J9 to J13, J16 to J14, J17 to J15, J18 to J16, J19 to J17, J20 to J19, J11 to J22, J12 to J23, J13 to J24, J14 to J25, J15 to J26, J8 to J7, J2 to P1
Connections:
- net CS_5V: now also J29.1 (Pin_1)
- net EN: now also J6.1 (Pin_1)
- net GND: now also J2.2 (Pin_2), J3.2 (Pin_2), J32.2 (Pin_2), J33.2 (Pin_2), J34.2 (Pin_2), J35.2 (Pin_2), J4.2 (Pin_2), J5.2 (Pin_2)
- net GPIO43: now also J20.1 (Pin_1); no longer J19.1 (Pin_1), S1.4, S2.4, S3.4, U2.6
- net INT: now also J27.1 (Pin_1)
- net SDA: now also J18.1 (Pin_1), J31.1 (Pin_1)
- net SDA_EXT: now also J25.1 (Pin_1), S4.4
- net SDO/ADR_3V: now also J28.1 (Pin_1)
- net VBat: now also J2.1 (Pin_1), J3.1 (Pin_1), J4.1 (Pin_1), J5.1 (Pin_1); no longer J6.1 (Pin_1)
- net VCC_3V3: now also J8.1 (Pin_1)
- net VCC_3V3_MCU: now also J9.1 (Pin_1); no longer J21.1 (Pin_1), S1.1, S2.1, S3.1
- removed net 3Vo: S1.2, S2.2, S3.2
- net 5VIN: no longer names the net of U1.1
- new net: J35.1 (Pin_1), J39.1 (Pin_1)
- new net: J33.1 (Pin_1), J37.1 (Pin_1)
- new net: J32.1 (Pin_1), J36.1 (Pin_1)
- new net: J34.1 (Pin_1), J38.1 (Pin_1)
- new net SCL: J19.1 (Pin_1), J30.1 (Pin_1), S1.4, S2.4, S3.4, U2.6
- new net VCC_3V3_Sensors: J21.1 (Pin_1), S1.1, S2.1, S3.1
- no-connect marks 0 -> 4
Other:
- note added: "14.8V Nominal"
- note added: "ESC Signal Headers"
- note added: "MCU Board"
- note added: "MCU GPIO --> Conn_MCUtoESC_x --> Conn_ESC_SIG_x"
- note added: "Power Distribution Board"
- note added: "Sensors Board"
- moved on the sheet: J1, J10, J11, J12, J13, J14, J15, J16, J17, J19, J21, J22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

Commit message: separate main schematic from power-board
Parts:
- removed J1: Conn_Lipo_Battery, symbol Connector_Generic:Conn_01x02
- removed J2: Conn_ESC_PWR_1, symbol Connector_Generic:Conn_01x02
- removed J3: Conn_ESC_PWR_2, symbol Connector_Generic:Conn_01x02
- removed J4: Conn_ESC_PWR_3, symbol Connector_Generic:Conn_01x02
- removed J5: Conn_ESC_PWR_4, symbol Connector_Generic:Conn_01x02
- removed P1: AF-MPM3610-Converter, Adafruit MPM3610:1X04_ROUND, symbol Adafruit MPM3610-eagle-import:HEADER-1X4ROUND
- removed S1: AF-QMC5883P-Magnetometer, Adafruit QMC5883P Magnetometer:1X05_ROUND_70, symbol Adafruit QMC5883P Magnetometer-eagle-import:HEADER-1X570MIL
- removed S2: AF-BMP280-Barometer, Adafruit BMP280:1X07_ROUND_70, symbol Adafruit BMP280-eagle-import:HEADER-1X770MIL
- removed S3: AF-MPU6050-Accel/Gyro, Adafruit MPU6050:1X06_ROUND_70, symbol Adafruit MPU6050-eagle-import:HEADER-1X670MIL
- removed S4: AF-MPU6050-Accel/Gyro, Adafruit MPU6050:1X06_ROUND, symbol Adafruit MPU6050-eagle-import:HEADER-1X6ROUND
- removed U1: ----Seeed-XIAO-ESP32-S3-Module----, symbol Adafruit BMP280-eagle-import:HEADER-1X770MIL
- removed U2: ESP32-S3, symbol Adafruit BMP280-eagle-import:HEADER-1X770MIL
- added H1, H2, H3, H4: MountingHole, MountingHole:MountingHole_3.2mm_M3_ISO14580_Pad_TopOnly, symbol Mechanical:MountingHole
- added J10: ESC_3_+, Solder_Pads:01x01_ESC_Pad_Vias, symbol Connector_Generic:Conn_01x01
- added J6: ESC_3_-, Solder_Pads:01x01_ESC_Pad, symbol Connector_Generic:Conn_01x01
- added J6: ESC_1_+, Solder_Pads:01x01_ESC_Pad_Vias, symbol Connector_Generic:Conn_01x01
- added J7: ESC_1_-, Solder_Pads:01x01_ESC_Pad, symbol Connector_Generic:Conn_01x01
- added J7: ESC_4_+, Solder_Pads:01x01_ESC_Pad_Vias, symbol Connector_Generic:Conn_01x01
- added J8: ESC_4_-, Solder_Pads:01x01_ESC_Pad, symbol Connector_Generic:Conn_01x01
- added J8: ESC_2_+, Solder_Pads:01x01_ESC_Pad_Vias, symbol Connector_Generic:Conn_01x01
- added J9: ESC_2_-, Solder_Pads:01x01_ESC_Pad, symbol Connector_Generic:Conn_01x01
- added J9: Conn_01x02, Solder_Pads:PDB_Battery_Pads_ViasL, symbol Connector_Generic:Conn_01x02
- added P1: AF-MPM3610-Converter, Connector_PinSocket_2.54mm:PinSocket_1x04_P2.54mm_Vertical, symbol Connector_Generic:Conn_01x04
- added S1: AF-MPU6050-Accel/Gyro-L, symbol Connector_Generic:Conn_01x06
- added S2: AF-MPU6050-Accel/Gyro-R, symbol Connector_Generic:Conn_01x06
- added S3: AF-BMP280-Barometer, symbol Connector_Generic:Conn_01x07
- added S4: AF-QMC5883P-Magnetometer, symbol Connector_Generic:Conn_01x05
- added U1: Seeed-XIAO-ESP32-S3-Module-L, Connector_PinSocket_2.54mm:PinSocket_1x07_P2.54mm_Vertical, symbol Connector_Generic:Conn_01x07
- added U2: Seeed-XIAO-ESP32-S3-Module-R, Connector_PinSocket_2.54mm:PinSocket_1x07_P2.54mm_Vertical, symbol Connector_Generic:Conn_01x07
- J1: renamed from J22; footprint (none) -> Connector_Wire:SolderWire-0.1sqmm_1x01_D0.4mm_OD1mm
- J10: renamed from J6; footprint (none) -> Connector_Wire:SolderWire-0.1sqmm_1x01_D0.4mm_OD1mm
- J11: renamed from J7; footprint (none) -> Connector_Wire:SolderWire-0.1sqmm_1x01_D0.4mm_OD1mm
- J12: renamed from J8; footprint (none) -> Connector_Wire:SolderWire-0.1sqmm_1x01_D0.4mm_OD1mm
- J14: renamed from J27; footprint (none) -> Connector_Wire:SolderWire-0.1sqmm_1x01_D0.4mm_OD1mm
- J15: renamed from J28; footprint (none) -> Connector_Wire:SolderWire-0.1sqmm_1x01_D0.4mm_OD1mm
- J16: renamed from J29; footprint (none) -> Connector_Wire:SolderWire-0.1sqmm_1x01_D0.4mm_OD1mm
- J18: renamed from J30; footprint (none) -> Connector_Wire:SolderWire-0.1sqmm_1x01_D0.4mm_OD1mm
- J2: renamed from J23; footprint (none) -> Connector_Wire:SolderWire-0.1sqmm_1x01_D0.4mm_OD1mm
- J22: renamed from J31; footprint (none) -> Connector_Wire:SolderWire-0.1sqmm_1x01_D0.4mm_OD1mm
- J23: renamed from J21; footprint (none) -> Connector_Wire:SolderWire-0.1sqmm_1x01_D0.4mm_OD1mm
- J24: renamed from J14; footprint (none) -> Connector_Wire:SolderWire-0.1sqmm_1x01_D0.4mm_OD1mm
- J25: renamed from J15; footprint (none) -> Connector_Wire:SolderWire-0.1sqmm_1x01_D0.4mm_OD1mm
- J26: renamed from J16; footprint (none) -> Connector_Wire:SolderWire-0.1sqmm_1x01_D0.4mm_OD1mm
- J27: renamed from J17; footprint (none) -> Connector_Wire:SolderWire-0.1sqmm_1x01_D0.4mm_OD1mm
- J28: renamed from J18; footprint (none) -> Connector_Wire:SolderWire-0.1sqmm_1x01_D0.4mm_OD1mm
- J29: renamed from J19; footprint (none) -> Connector_Wire:SolderWire-0.1sqmm_1x01_D0.4mm_OD1mm
- J3: renamed from J24; footprint (none) -> Connector_Wire:SolderWire-0.1sqmm_1x01_D0.4mm_OD1mm
- J30: renamed from J20; footprint (none) -> Connector_Wire:SolderWire-0.1sqmm_1x01_D0.4mm_OD1mm
- J31: renamed from J36; footprint (none) -> Connector_Wire:SolderWire-0.1sqmm_1x01_D0.4mm_OD1mm
- J32: renamed from J37; footprint (none) -> Connector_Wire:SolderWire-0.1sqmm_1x01_D0.4mm_OD1mm
- J33: renamed from J38; footprint (none) -> Connector_Wire:SolderWire-0.1sqmm_1x01_D0.4mm_OD1mm
- J34: renamed from J39; footprint (none) -> Connector_Wire:SolderWire-0.1sqmm_1x01_D0.4mm_OD1mm
- J35: renamed from J9; footprint (none) -> Connector_Wire:SolderWire-0.1sqmm_1x01_D0.4mm_OD1mm
- J36: renamed from J10; footprint (none) -> Connector_Wire:SolderWire-0.1sqmm_1x01_D0.4mm_OD1mm
- J37: renamed from J11; footprint (none) -> Connector_Wire:SolderWire-0.1sqmm_1x01_D0.4mm_OD1mm
- J38: renamed from J32; footprint (none) -> Connector_Wire:SolderWire-0.1sqmm_1x02_P3.6mm_D0.4mm_OD1mm
- J39: renamed from J33; footprint (none) -> Connector_Wire:SolderWire-0.1sqmm_1x02_P3.6mm_D0.4mm_OD1mm
- J4: renamed from J25; footprint (none) -> Connector_Wire:SolderWire-0.1sqmm_1x01_D0.4mm_OD1mm
- J40: renamed from J34; footprint (none) -> Connector_Wire:SolderWire-0.1sqmm_1x02_P3.6mm_D0.4mm_OD1mm
- J41: renamed from J35; footprint (none) -> Connector_Wire:SolderWire-0.1sqmm_1x02_P3.6mm_D0.4mm_OD1mm
- J42: renamed from J12; footprint (none) -> Connector_Wire:SolderWire-0.1sqmm_1x01_D0.4mm_OD1mm
- J43: renamed from J13; footprint (none) -> Connector_Wire:SolderWire-0.1sqmm_1x01_D0.4mm_OD1mm
- J5: renamed from J26; footprint (none) -> Connector_Wire:SolderWire-0.1sqmm_1x01_D0.4mm_OD1mm
Connections:
- net AD0: now also S1.1 (Pin_1)
- net CLKIN: now also S1.5 (Pin_5)
- net CS_5V: now also S3.7 (Pin_7)
- net EN: now also P1.1 (Pin_1)
- net FSYNC_IN: now also S1.2 (Pin_2)
- net GND: now also J6.1 (Pin_1), J7.1 (Pin_1), J8.1 (Pin_1), J9.1 (Pin_1), J9.2 (Pin_2), P1.4 (Pin_4), S1.6 (Pin_6), S2.3 (Pin_3), S3.3 (Pin_3), S4.3 (Pin_3), U2.2 (Pin_2)
- net GPIO1: now also U1.1 (Pin_1)
- net GPIO2: now also U1.2 (Pin_2)
- net GPIO3: now also U1.3 (Pin_3)
- net GPIO4: now also U1.4 (Pin_4)
- net GPIO43: now also U1.7 (Pin_7)
- net GPIO44: now also U2.7 (Pin_7)
- net GPIO7: now also U2.6 (Pin_6)
- net GPIO8: now also U2.5 (Pin_5)
- net GPIO9: now also U2.4 (Pin_4)
- net INT: now also S2.6 (Pin_6)
- net SCL: now also S2.4 (Pin_4), S3.4 (Pin_4), S4.4 (Pin_4), U1.6 (Pin_6)
- net SCL_EXT: now also S1.3 (Pin_3)
- net SDA: now also S2.5 (Pin_5), S3.6 (Pin_6), S4.5 (Pin_5), U1.5 (Pin_5)
- net SDA_EXT: now also S1.4 (Pin_4)
- net SDO/ADR_3V: now also S3.5 (Pin_5)
- net VBat: now also J10.1 (Pin_1), J6.1 (Pin_1), J7.1 (Pin_1), J8.1 (Pin_1), J9.1 (Pin_1), P1.2 (Pin_2)
- net VCC_3V3: now also P1.3 (Pin_3)
- net VCC_3V3_MCU: now also U2.3 (Pin_3)
- net VCC_3V3_Sensors: now also S2.1 (Pin_1), S3.1 (Pin_1), S4.1 (Pin_1)
Other:
- moved on the sheet: J10, J11, J12
